File: Schematic/Schematic nhom1.kicad_sch (KiCad schematic)
At the start: 17 parts, among them K2 Fujitsu_FTR-LYCA005x, Q1 BC547, U1 ATmega328-P

Commit message: push schemactic
Parts:
- removed V1: VSIN, symbol Simulation_SPICE:VSIN
- added V2: 1, symbol Simulation_SPICE:VDC
- renumbered LM1 to LM2596
Connections:
- net at LM2596.1 (IN-): now also V2.2
- net at LM2596.2 (IN+): now also V2.1
Changed lines of the file:
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@@
+	)
+	(symbol
+		(lib_id "Simulation_SPICE:VDC")
+		(at 212.09 74.93 270)
+		(unit 1)
+		(exclude_from_sim no)
+		(in_bom yes)
+		(on_board yes)
+		(dnp no)
+		(fields_autoplaced yes)
+		(property "Reference" "V2"
+			(at 212.2198 67.31 90)
+			(effects
+				(font
+					(size 1.27 1.27)
+				)
+			)
+		)
+		(property "Value" "1"
+			(at 212.2198 69.85 90)
+			(effects
+				(font
+					(size 1.27 1.27)
+				)
+			)
+		)
+		(property "Footprint" ""
+			(at 212.09 74.93 0)
+			(effects
+				(font
+					(size 1.27 1.27)
+				)
+				(hide yes)
+			)
+		)
+		(property "Datasheet" "https://ngspice.sourceforge.io/docs/ngspice-html-manual/manual.xhtml#sec_Independent_Sources_for"
+			(at 212.09 74.93 0)
+			(effects
+				(font
+					(size 1.27 1.27)
+				)
+				(hide yes)
+			)
+		)
+		(property "Description" "Voltage source, DC"
+			(at 212.09 74.93 0)
+			(effects
+				(font
+					(size 1.27 1.27)
+				)
+				(hide yes)
+			)
+		)
+		(property "Sim.Pins" "1=+ 2=-"
+			(at 212.09 74.93 0)
+			(effects
+				(font
+					(size 1.27 1.27)
+				)
+				(hide yes)
+			)
+		)
+		(property "Sim.Type" "DC"
+			(at 212.09 74.93 0)
+			(effects
+				(font
+					(size 1.27 1.27)
+				)
+				(hide yes)
+			)
+		)
+		(property "Sim.Device" "V"
+			(at 212.09 74.93 0)
+			(effects
+				(font
+					(size 1.27 1.27)
+				)
+				(justify left)
+				(hide yes)
+			)
+		)
+		(pin "1"
+		)
+		(pin "2"
+		)
+		(instances
+			(project ""
+				(path "/23bca959-424d-432f-8902-aec505b99b2a"
+					(reference "V2")
+					(unit 1)
+				)
+			)
+		)
 	)
 	(symbol
@@
 		(dnp no)
 		(fields_autoplaced yes)
-		(property "Reference" "LM1"
+		(property "Reference" "LM2596"
 			(at 218.44 99.0599 0)
 			(effects
@@
 			(project ""
 				(path "/23bca959-424d-432f-8902-aec505b99b2a"
-					(reference "LM1")
+					(reference "LM2596")
 					(unit 1)
 				)
@@
 					(unit 1)
 				)
-			)
-		)
-	)
-	(symbol
-		(lib_id "Simulation_SPICE:VSIN")
-		(at 212.09 74.93 270)
-		(unit 1)
-		(exclude_from_sim no)
-		(in_bom yes)
-		(on_board yes)
-		(dnp no)
-		(fields_autoplaced yes)
-		(property "Reference" "V1"
-			(at 212.2198 64.77 90)
-			(effects
-				(font
-					(size 1.27 1.27)
-				)
-			)
-		)
-		(property "Value" "VSIN"
-			(at 212.2198 67.31 90)
-			(effects
-				(font
-					(size 1.27 1.27)
-				)
-			)
-		)
-		(property "Footprint" ""
-			(at 212.09 74.93 0)
-			(effects
-				(font
-					(size 1.27 1.27)
-				)
-				(hide yes)
-			)
-		)
-		(property "Datasheet" "https://ngspice.sourceforge.io/docs/ngspice-html-manual/manual.xhtml#sec_Independent_Sources_for"
-			(at 212.09 74.93 0)
-			(effects
-				(font
-					(size 1.27 1.27)
-				)
-				(hide yes)
-			)
-		)
-		(property "Description" "Voltage source, sinusoidal"
-			(at 212.09 74.93 0)
-			(effects
-				(font
-					(size 1.27 1.27)
-				)
-				(hide yes)
-			)
-		)
-		(property "Sim.Pins" "1=+ 2=-"
-			(at 212.09 74.93 0)
-			(effects
-				(font
-					(size 1.27 1.27)
-				)
-				(hide yes)
-			)
-		)
-		(property "Sim.Params" "dc=0 ampl=1 f=1k ac=1"
-			(at 212.2198 69.85 90)
-			(effects
-				(font
-					(size 1.27 1.27)
-				)
-			)
-		)
-		(property "Sim.Type" "SIN"
-			(at 212.09 74.93 0)
-			(effects
-				(font
-					(size 1.27 1.27)
-				)
-				(hide yes)
-			)
-		)
-		(property "Sim.Device" "V"
-			(at 212.09 74.93 0)
-			(effects
-				(font
-					(size 1.27 1.27)
-				)
-				(justify left)
-				(hide yes)
-			)
-		)
-		(pin "1"
-		)
-		(pin "2"
-		)
-		(instances
-			(project ""
-				(path "/23bca959-424d-432f-8902-aec505b99b2a"
-					(reference "V1")
-					(unit 1)
-				)

Commit message: Summary Schematic
Parts:
- removed V2: 1, symbol Simulation_SPICE:VDC
- added BT1: Battery, symbol Device:Battery
- added SW1: SW_Push, symbol Switch:SW_Push
Connections:
- net at LM2596.2 (IN+): now also BT1.1 (+)
- net at LM2596.1 (IN-): now also BT1.2 (-)
- net at R4.1: now also SW1.1
Changed lines of the file:
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@@
+	)
+	(junction
+		(at 109.22 140.97)
+		(diameter 0)
+		(color 0 0 0 0)
 	)
 	(junction
@@
 	(wire
 		(pts
+			(xy 109.22 137.16) (xy 109.22 140.97)
+		)
+		(stroke
+			(width 0)
+			(type default)
+		)
+	)
+	(wire
+		(pts
 			(xy 95.25 96.52) (xy 95.25 101.6)
 		)
@@
 	(wire
 		(pts
+			(xy 109.22 140.97) (xy 102.87 140.97)
+		)
+		(stroke
+			(width 0)
+			(type default)
+		)
+	)
+	(wire
+		(pts
 			(xy 90.17 140.97) (xy 95.25 140.97)
 		)
@@
 	(wire
 		(pts
+			(xy 109.22 140.97) (xy 127 140.97)
+		)
+		(stroke
+			(width 0)
+			(type default)
+		)
+	)
+	(wire
+		(pts
 			(xy 87.63 113.03) (xy 93.98 113.03)
 		)
@@
 	(wire
 		(pts
+			(xy 109.22 121.92) (xy 109.22 127)
+		)
+		(stroke
+			(width 0)
+			(type default)
+		)
+	)
+	(wire
+		(pts
 			(xy 95.25 93.98) (xy 143.51 93.98)
 		)
@@
 	(wire
 		(pts
-			(xy 102.87 140.97) (xy 110.49 140.97)
-		)
-		(stroke
-			(width 0)
-			(type default)
-		)
-	)
-	(wire
-		(pts
 			(xy 88.265 85.09) (xy 88.265 81.915)
 		)
@@
 		)
 	)
+	(text "1"
+		(exclude_from_sim no)
+		(at 124.968 139.7 0)
+		(effects
+			(font
+				(size 1.27 1.27)
+			)
+		)
+	)
 	(text "GND"
 		(exclude_from_sim no)
@@
 		)
 	)
-	(text "1"
-		(exclude_from_sim no)
-		(at 109.22 138.938 0)
+	(text "GND"
+		(exclude_from_sim no)
+		(at 111.76 124.968 0)
 		(effects
 			(font
@@
 	)
 	(symbol
-		(lib_id "Simulation_SPICE:VDC")
-		(at 212.09 74.93 270)
-		(unit 1)
-		(exclude_from_sim no)
-		(in_bom yes)
-		(on_board yes)
-		(dnp no)
-		(fields_autoplaced yes)
-		(property "Reference" "V2"
-			(at 212.2198 67.31 90)
-			(effects
-				(font
-					(size 1.27 1.27)
-				)
-			)
-		)
-		(property "Value" "1"
-			(at 212.2198 69.85 90)
-			(effects
-				(font
-					(size 1.27 1.27)
-				)
-			)
-		)
-		(property "Footprint" ""
-			(at 212.09 74.93 0)
-			(effects
-				(font
-					(size 1.27 1.27)
-				)
-				(hide yes)
-			)
-		)
-		(property "Datasheet" "https://ngspice.sourceforge.io/docs/ngspice-html-manual/manual.xhtml#sec_Independent_Sources_for"
-			(at 212.09 74.93 0)
-			(effects
-				(font
-					(size 1.27 1.27)
-				)
-				(hide yes)
-			)
-		)
-		(property "Description" "Voltage source, DC"
-			(at 212.09 74.93 0)
-			(effects
-				(font
-					(size 1.27 1.27)
-				)
-				(hide yes)
-			)
-		)
-		(property "Sim.Pins" "1=+ 2=-"
-			(at 212.09 74.93 0)
-			(effects
-				(font
-					(size 1.27 1.27)
-				)
-				(hide yes)
-			)
-		)
-		(property "Sim.Type" "DC"
-			(at 212.09 74.93 0)
-			(effects
-				(font
-					(size 1.27 1.27)
-				)
-				(hide yes)
-			)
-		)
-		(property "Sim.Device" "V"
-			(at 212.09 74.93 0)
-			(effects
-				(font
-					(size 1.27 1.27)
-				)
-				(justify left)
-				(hide yes)
-			)
-		)
-		(pin "1"
-		)
-		(pin "2"
-		)
-		(instances
-			(project ""
-				(path "/23bca959-424d-432f-8902-aec505b99b2a"
-					(reference "V2")
-					(unit 1)
-				)
-			)
-		)
-	)
-	(symbol
 		(lib_id "Device:R")
 		(at 80.01 69.85 270)
@@
 	)
 	(symbol
+		(lib_id "Switch:SW_Push")
+		(at 109.22 132.08 90)
+		(unit 1)
+		(exclude_from_sim no)
+		(in_bom yes)
+		(on_board yes)
+		(dnp no)
+		(fields_autoplaced yes)
+		(property "Reference" "SW1"
+			(at 110.49 130.8099 90)
+			(effects
+				(font
+					(size 1.27 1.27)
+				)
+				(justify right)
+			)
+		)
+		(property "Value" "SW_Push"
+			(at 110.49 133.3499 90)
+			(effects
+				(font
+					(size 1.27 1.27)
+				)
+				(justify right)
+			)
+		)
+		(property "Footprint" ""
+			(at 104.14 132.08 0)
+			(effects
+				(font
+					(size 1.27 1.27)
+				)
+				(hide yes)
+			)
+		)
+		(property "Datasheet" "~"
+			(at 104.14 132.08 0)
+			(effects
+				(font
+					(size 1.27 1.27)
+				)
+				(hide yes)
+			)
+		)
+		(property "Description" "Push button switch, generic, two pins"
+			(at 109.22 132.08 0)
+			(effects
+				(font
+					(size 1.27 1.27)
+				)
+				(hide yes)
+			)
+		)
+		(pin "2"
+		)
+		(pin "1"
+		)
+		(instances
+			(project ""
+				(path "/23bca959-424d-432f-8902-aec505b99b2a"
+					(reference "SW1")
+					(unit 1)
+				)
+			)
+		)
+	)
+	(symbol
 		(lib_id "Relay:Fujitsu_FTR-LYCA005x")
 		(at 52.07 77.47 180)
@@
 					(unit 1)
 				)
+			)
+		)
+	)
+	(symbol
+		(lib_id "Device:Battery")
+		(at 212.09 74.93 270)
+		(unit 1)
+		(exclude_from_sim no)
+		(in_bom yes)
+		(on_board yes)
+		(dnp no)
+		(fields_autoplaced yes)
+		(property "Reference" "BT1"
+			(at 212.6615 67.31 90)
+			(effects
+				(font
+					(size 1.27 1.27)
+				)
+			)
+		)
+		(property "Value" "Battery"
+			(at 212.6615 69.85 90)
+			(effects
+				(font
+					(size 1.27 1.27)
+				)
+			)
+		)
+		(property "Footprint" ""
+			(at 213.614 74.93 90)
+			(effects
+				(font
+					(size 1.27 1.27)
+				)
+				(hide yes)
+			)
+		)
+		(property "Datasheet" "~"
+			(at 213.614 74.93 90)
+			(effects
+				(font
+					(size 1.27 1.27)
+				)
+				(hide yes)
+			)
+		)
+		(property "Description" "Multiple-cell battery"
+			(at 212.09 74.93 0)
+			(effects
+				(font
+					(size 1.27 1.27)
+				)
+				(hide yes)
+			)
+		)
+		(pin "2"
+		)
+		(pin "1"
+		)
+		(instances
+			(project ""
+				(path "/23bca959-424d-432f-8902-aec505b99b2a"
+					(reference "BT1")
+					(unit 1)
+				)

Commit message: summit Schematic
Parts:
- removed GSM_Module1: SIM800L, symbol sim800l:SIM800L
- removed U1: ATmega328-P, Package_DIP:DIP-28_W7.62mm, symbol MCU_Microchip_ATmega:ATmega328-P
- added C4, C5: 10uF, symbol Device:C
- added D3: LED BAO NGUON, symbol Device:LED
- added GSM_Module2: SIM7680c, symbol SIM800L:SIM_A7680c
- added J1: AVR-ISP-6, symbol Connector:AVR-ISP-6
- added R5: 1K, symbol Device:R
- added U1: ~, symbol MCU_Microchip_ATmega 328P:atmega328p
Connections:
- net Earth: now reaches C1.1, C2.1, C3.2
- net Earth: now also LM2596.3 (OUT-), Q1.3 (E), R3.2, SW1.2, U3.4 (GND), C4.2, C5.2, D3.1 (K), GSM_Module2.6 (GND), J1.6 (GND), U1.22 (GND), U1.8 (GND)
- net VCC: now reaches LM2596.4 (OUT+)
- net VCC: now also U3.1 (VCC), C5.1, J1.2 (VCC), R5.1, U1.20 (AVCC), U1.7 (VCC)
- net at R4.2: no longer U3.1 (VCC)
- new net: D3.2 (A), R5.2
- new net: C4.1, U1.21 (AREF)
Other:
- note added: "ATMEGA 328P"
- note added: "Hệ thống điều khiển động cơ xe máy"
- note added: "KHOI NAP"
- note added: "KHOI NGUON"
- note added: "MISO"
- note added: "MODULE GPS"
- note added: "MODULE SIM"
- note added: "MOSI"
- note added: "NGAT DONG CO XE"
- note added: "PB0"
- note added: "PB1"
- note added: "PB4"
- note added: "PD2"
- note added: "PD3"
- note added: "RESET"
- note added: "SCK"
- note added: "SWITCH"
- note added: "THACH ANH"
- note added: "XTAL1"
- note added: "XTAL2"
- note added: "sim net"
- note added: "vcc gps"
- note removed: "1"
- note removed: "14"
- note removed: "15"
- note removed: "18"
- note removed: "22"
- note removed: "4"
- note removed: "5"
- moved on the sheet: BT1, C3, D1, D2, LM2596, Q1, R1, R2, R3, R4, U3
